File: liberation/liberation.kicad_pcb (KiCad board)
At the start: 2 copper layers, 71.1 x 69.8 mm, 21 parts, among them Q1 BC547BTA, Q2 BC547BTA, SW1 MHS122K, SW2 FSM4JAH, U1 NJU7223F33, U2 ESP32-WROOM-32D, U3 BME280

Commit message: Make PCB design (almost) complete :p
Parts:
- removed BT1: Battery, Battery:keystone_2477
- moved C4 64.8 mm to (134.0, 91.4), turned to 180 degrees
- moved SW1 62.1 mm to (98.4, 124.8), turned to 0 degrees
- moved C1 61.0 mm to (142.2, 135.9)
- moved R7 57.3 mm to (149.9, 88.9)
- moved R6 56.6 mm to (149.9, 95.2)
- moved U3 54.4 mm to (122.6, 91.4), turned to 180 degrees
- moved R1 50.1 mm to (149.9, 127.0), turned to 180 degrees
- moved U1 28.9 mm to (116.2, 130.4), turned to 270 degrees
- moved C2 20.1 mm to (125.7, 135.9), turned to 0 degrees
- moved R5 18.2 mm to (142.2, 108.0)
- moved U2 17.8 mm to (108.0, 95.2)
- moved Q1 17.7 mm to (131.4, 113.0)
- moved Q2 17.7 mm to (131.4, 119.4)
- moved R8 17.2 mm to (106.7, 116.2), turned to 180 degrees
- moved R4 16.9 mm to (142.2, 101.6)
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Connections:
- Jserial1 pad 2: RTS -> DTR
- Jserial1 pad 3: DTR -> RTS
- SW1 pad 1: Net-(BT1-Pad1) -> (no net)
- U1 pad 1: VBAT -> +3V3
- U1 pad 2: GND -> VBAT
- U1 pad 3: +3V3 -> GND
- U2 pad 10: Net-(U2-Pad10) -> (no net)
- U2 pad 11: Net-(U2-Pad11) -> (no net)
- U2 pad 12: Net-(U2-Pad12) -> (no net)
- U2 pad 13: Net-(U2-Pad13) -> (no net)
- U2 pad 14: Net-(U2-Pad14) -> (no net)
- U2 pad 17: Net-(U2-Pad17) -> (no net)
- U2 pad 18: Net-(U2-Pad18) -> (no net)
- U2 pad 19: Net-(U2-Pad19) -> (no net)
- U2 pad 20: Net-(U2-Pad20) -> (no net)
- U2 pad 21: Net-(U2-Pad21) -> (no net)
- U2 pad 22: Net-(U2-Pad22) -> (no net)
- U2 pad 23: Net-(U2-Pad23) -> (no net)
- U2 pad 24: Net-(U2-Pad24) -> (no net)
- U2 pad 26: Net-(U2-Pad26) -> (no net)
- U2 pad 27: Net-(U2-Pad27) -> (no net)
- U2 pad 28: Net-(U2-Pad28) -> (no net)
- U2 pad 29: Net-(U2-Pad29) -> (no net)
- U2 pad 30: Net-(U2-Pad30) -> (no net)
- U2 pad 31: Net-(U2-Pad31) -> (no net)
- U2 pad 37: Net-(U2-Pad37) -> (no net)
- U2 pad 4: Net-(U2-Pad4) -> (no net)
- U2 pad 5: Net-(U2-Pad5) -> (no net)
- U2 pad 6: Net-(U2-Pad6) -> (no net)
- U2 pad 7: Net-(U2-Pad7) -> (no net)
- U2 pad 8: Net-(U2-Pad8) -> (no net)
- U2 pad 9: Net-(U2-Pad9) -> (no net)
Routing:
- net +3V3: track 153.3 -> 222.0 mm
- net SCL: track 50.2 -> 27.3 mm, vias 1 -> 0
- net Net-(R5-Pad1): track 13.8 -> 31.1 mm
- net Net-(BT1-Pad1): track 17.1 -> 0.00 mm
- net GND: track 0.00 -> 16.2 mm, vias 0 -> 18
- net SDA: track 50.8 -> 35.8 mm, vias 1 -> 2
- net RTS: track 27.0 -> 41.3 mm, vias 0 -> 2
- net Net-(R4-Pad1): track 15.4 -> 29.0 mm
- net RESET: track 60.1 -> 72.7 mm
- net TXD: track 7.62 -> 16.6 mm
- net Net-(Q2-Pad2): track 5.08 -> 10.8 mm
- net Net-(Q1-Pad2): track 5.08 -> 10.8 mm
- net DTR: track 50.4 -> 44.7 mm
- net BOOT: track 14.1 -> 17.9 mm
- net RXD: track 9.42 -> 12.8 mm
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- added copper zone on B.Cu, net GND
Other:
- board size 71.1 x 69.8 mm -> 66.7 x 69.8 mm

Commit message: finich pcb and secmatic for ordering
Parts:
- added BT1: Battery, Battery:keystone_2477, B.Cu at (150.9, 149.4)
- added G***: LOGO, logo:rheon, F.Cu at (122.6, 107.3)
- added G***: LOGO, logo:hhs-logo, F.Cu at (131.4, 102.5)
- U1: footprint Package_TO_SOT_THT:TO-3P-3_Vertical -> Package_TO_SOT_THT:NJU7223F33
- renumbered Q2 to Q1, Q1 to Q2, R3 to R2, R2 to R3, R5 to R4, R4 to R5
Connections:
- SW1 pad 1: (no net) -> Net-(BT1-Pad1)
- U1 pad 1: +3V3 -> VBAT
- U1 pad 2: VBAT -> GND
- U1 pad 3: GND -> +3V3
- U2 pad 10: (no net) -> Net-(U2-Pad10)
- U2 pad 11: (no net) -> Net-(U2-Pad11)
- U2 pad 12: (no net) -> Net-(U2-Pad12)
- U2 pad 13: (no net) -> Net-(U2-Pad13)
- U2 pad 14: (no net) -> Net-(U2-Pad14)
- U2 pad 17: (no net) -> Net-(U2-Pad17)
- U2 pad 18: (no net) -> Net-(U2-Pad18)
- U2 pad 19: (no net) -> Net-(U2-Pad19)
- U2 pad 20: (no net) -> Net-(U2-Pad20)
- U2 pad 21: (no net) -> Net-(U2-Pad21)
- U2 pad 22: (no net) -> Net-(U2-Pad22)
- U2 pad 23: (no net) -> Net-(U2-Pad23)
- U2 pad 24: (no net) -> Net-(U2-Pad24)
- U2 pad 26: (no net) -> Net-(U2-Pad26)
- U2 pad 27: (no net) -> Net-(U2-Pad27)
- U2 pad 28: (no net) -> Net-(U2-Pad28)
- U2 pad 29: (no net) -> Net-(U2-Pad29)
- U2 pad 30: (no net) -> Net-(U2-Pad30)
- U2 pad 31: (no net) -> Net-(U2-Pad31)
- U2 pad 37: (no net) -> Net-(U2-Pad37)
- U2 pad 4: (no net) -> Net-(U2-Pad4)
- U2 pad 5: (no net) -> Net-(U2-Pad5)
- U2 pad 6: (no net) -> Net-(U2-Pad6)
- U2 pad 7: (no net) -> Net-(U2-Pad7)
- U2 pad 8: (no net) -> Net-(U2-Pad8)
- U2 pad 9: (no net) -> Net-(U2-Pad9)
Routing:
- net Net-(BT1-Pad1): track 0.00 -> 60.3 mm
- net +3V3: track 222.0 -> 213.1 mm
Other:
- board text added: "+3V3"
- board text added: "Battery Holder"
- board text added: "By: Bob Swinkels & Luca van Straaten"
- board text added: "DTR"
- board text added: "GND"
- board text added: "JLCJLCJLCJLC"
- board text added: "Power Switch"
- board text added: "RTS"
- board text added: "RXD"
- board text added: "TXD"
- board text added: "WOW Monitor"
- board text added: "v1.0"
- board text removed: "ON/OFF Switch"
